File: Voltera Project Gerbers/Drill Tutorial Circuit/Punk_Console.brd (EAGLE design)
At the start: 14 parts, among them IC1 NE556D

Commit message: Updated Punk Console circuit
Parts:
- removed U$2, U$3: VOLT_RIVET1MM, voltera:VOLT_RIVET_1MM
- added U$5: BUZZER, voltera:BUZZER_PS1240P02BT
- moved C1 14.6 mm to (24.1, 12.3)
Connections:
- net MIC: now also U$5.P$2; no longer U$3.P$1
- net VCC: now also U$5.P$1; no longer U$2.P$1
Routing:
- net THR1: track 48.6 -> 35.1 mm
- net VCC: track 65.0 -> 69.2 mm
- net GND: track 78.2 -> 81.1 mm
Other:
- board text added: "556"
- board text added: "BUZZER"
- board text added: "LED"
- board text added: "TRIMPOT"
