File: Voltera Template Gerbers/2x3/2x3.brd (EAGLE design)
At the start: 76.2 x 50.8 mm, 1 part

Commit message: Created FAB version for evertying, removed bad versions
Parts:
- removed E$1: (no value), voltera_community_lib:2X3_BOARD
- added E$2: (no value), voltera_EAGLE_community_lib:2X3_BOARD
Changed lines of the file:
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@@
 <?xml version="1.0" encoding="utf-8"?>
 <!DOCTYPE eagle SYSTEM "eagle.dtd">
-<eagle version="7.6.0">
+<eagle version="8.7.0">
 <drawing>
 <settings>
 <setting alwaysvectorfont="no"/>
+<setting keepoldvectorfont="yes"/>
 <setting verticaltext="up"/>
 </settings>
@@
 <param name="dpMaxLengthDifference" value="10mm"/>
 <param name="dpGapFactor" value="2.5"/>
-<param name="checkGrid" value="0"/>
 <param name="checkAngle" value="0"/>
 <param name="checkFont" value="1"/>
 <param name="checkRestrict" value="1"/>
+<param name="checkStop" value="0"/>
+<param name="checkValues" value="0"/>
 <param name="useDiameter" value="13"/>
 <param name="maxErrors" value="50"/>
@@
 </autorouter>
 <elements>
-<element name="E$1" library="voltera_community_lib" package="2X3_BOARD" value="" x="0" y="0"/>
+<element name="E$2" library="voltera_EAGLE_community_lib" package="2X3_BOARD" value="" x="0" y="0"/>
 </elements>
 <signals>
